File: V1/RJ45-breakout_8ch-V1.kicad_pcb (KiCad board)
At the start: 2 copper layers, 173 x 67.8 mm, 17 parts, among them J1 RJ45, J10 Screw_Terminal_01x04, J11 Screw_Terminal_01x04, J12 Screw_Terminal_01x04, J13 Screw_Terminal_01x04, J14 Screw_Terminal_01x04, J15 Screw_Terminal_01x04, J16 Screw_Terminal_01x04, J2 RJ45, J3 RJ45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

Commit message: updates to components
Other:
- net class Default removed
