File: V2/RJ45-breakout_8ch-V2.kicad_pcb (KiCad board)
At the start: 2 copper layers, 133 x 67.8 mm, 17 parts, among them J1 RJ45, J10 Screw_Terminal_01x03, J11 Screw_Terminal_01x03, J12 Screw_Terminal_01x03, J13 Screw_Terminal_01x03, J14 Screw_Terminal_01x03, J15 Screw_Terminal_01x03, J16 Screw_Terminal_01x03, J2 RJ45, J3 RJ45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

Commit message: PCB tweaks
Parts:
- removed the REF** at (95.2, 69.8)
- added ?: , Tales:TMaschio_20x6.4mm, F.Cu at (157.5, 66.0)
- added REF**: OSHW-Logo2_14.6x12mm_SilkScreen, Symbol:OSHW-Logo2_14.6x12mm_SilkScreen, F.Cu at (215.9, 68.6)
- moved J12 27.1 mm to (148.0, 114.3)
- moved J14 27.1 mm to (178.4, 114.3)
- moved J15 27.1 mm to (193.7, 114.3)
- moved J3 27.1 mm to (132.1, 78.7)
- moved J5 27.1 mm to (162.6, 78.7)
- moved J6 27.1 mm to (177.8, 97.8)
- moved J11 27.1 mm to (132.7, 114.3)
- moved J2 27.1 mm to (116.8, 97.8)
- moved J9 27.1 mm to (97.2, 114.3)
- moved J1 27.1 mm to (101.6, 78.7)
- moved J10 27.1 mm to (117.5, 114.3)
- moved J13 27.1 mm to (163.2, 114.3)
- moved J16 27.1 mm to (208.9, 114.3)
- moved J4 27.1 mm to (147.3, 97.8)
- moved J7 27.1 mm to (193.0, 78.7)
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