File: V2/RJ45-breakout_8ch-V2.kicad_sch (KiCad schematic)
At the start: 16 parts, among them J1 RJ45, J10 Screw_Terminal_01x03, J11 Screw_Terminal_01x03, J12 Screw_Terminal_01x03, J13 Screw_Terminal_01x03, J14 Screw_Terminal_01x03, J15 Screw_Terminal_01x03, J16 Screw_Terminal_01x03, J2 RJ45, J3 RJ45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

Commit message: PCB tweaks
Other:
- title: (none) -> 8 channel RJ45 breakout board
Changed lines of the file:
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@@
 (kicad_sch (version 20211123) (generator eeschema)
   (paper "A4")
+  (title_block
+    (title "8 channel RJ45 breakout board")
+    (date "2022-04-01")
+    (rev "V2")
+  )
   (junction (at 91.44 80.01) (diameter 0) (color 0 0 0 0)
   )
