File: V2/RJ45-breakout-8ch-V2.kicad_pcb (KiCad board)
At the start: 2 copper layers, 133 x 67.8 mm, 18 parts, among them J1 RJ45, J10 Screw_Terminal_01x03, J11 Screw_Terminal_01x03, J12 Screw_Terminal_01x03, J13 Screw_Terminal_01x03, J14 Screw_Terminal_01x03, J15 Screw_Terminal_01x03, J16 Screw_Terminal_01x03, J2 RJ45, J3 RJ45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

Commit message: pcb tweaks
Other:
- board text added: "RJ45-BREAKOUT-8CH-V2"
Changed lines of the file:
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@@
     (effects (font (size 1.5 1.5) (thickness 0.25)))
+  )
+  (gr_text "RJ45-BREAKOUT-8CH-V2" (at 193.04 64.77) (layer "F.SilkS")
+    (effects (font (size 1.2 1.2) (thickness 0.2)))
   )
   (gr_text "CHANNEL 4" (at 151.13 88.265) (layer "F.SilkS")

Commit message: Update RJ45-breakout-8ch-V2.kicad_pcb
Parts:
- removed ?: , Tales:TMaschio_20x6.4mm
Other:
- board text added: "TMASCHIO 2022"
