File: V2/rj45-breakout-8ch-v2.kicad_pcb (KiCad board)
At the start: 2 copper layers, 133 x 67.8 mm, 17 parts, among them J1 RJ45, J10 Screw_Terminal_01x03, J11 Screw_Terminal_01x03, J12 Screw_Terminal_01x03, J13 Screw_Terminal_01x03, J14 Screw_Terminal_01x03, J15 Screw_Terminal_01x03, J16 Screw_Terminal_01x03, J2 RJ45, J3 RJ45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

Commit message: Update to Kicad 8
Parts:
- removed REF**: OSHW-Logo2_14.6x12mm_SilkScreen, Symbol:OSHW-Logo2_14.6x12mm_SilkScreen
