File: V3/rj45-breakout-8ch-v3.kicad_sch (KiCad schematic)
At the start: 13 parts, among them J1 Jack RJ45, J10 DB141V-2.54-6P, J11 DB141V-2.54-6P, J12 DB141V-2.54-6P, J13 DB141V-2.54-6P, J2 Jack RJ45, J3 Jack RJ45, J4 Jack RJ45, J5 Jack RJ45, J6 Jack RJ45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

Commit message: Update components
Other:
- title: 8 channel RJ45 breakout board -> 8 Channel RJ45 Breakout Board
Changed lines of the file:
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@@
 	(paper "A4")
 	(title_block
-		(title "8 channel RJ45 breakout board")
+		(title "8 Channel RJ45 Breakout Board")
 		(date "2022-04-01")
 		(rev "V3")

Commit message: Prefab checks
Parts:
- J9: footprint Tales:TerminalBlock_Dibo_DB142V-2-5.08_1x02_P5.08mm_Vertical -> Tales:TerminalBlock_Dibo_DB142V-5.08-2P_1x02_P5.08mm_Vertical
Changed lines of the file:
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@@
 			)
 		)
-		(property "Footprint" "Tales:TerminalBlock_Dibo_DB142V-2-5.08_1x02_P5.08mm_Vertical"
+		(property "Footprint" "Tales:TerminalBlock_Dibo_DB142V-5.08-2P_1x02_P5.08mm_Vertical"
 			(at 113.03 29.21 0)
 			(effects
