File: V3/rj45-breakout-8ch-v3.kicad_sch (KiCad schematic)
At the start: 13 parts, among them J1 Jack RJ45, J10 DB141V-2.54-6P, J11 DB141V-2.54-6P, J12 DB141V-2.54-6P, J13 DB141V-2.54-6P, J2 Jack RJ45, J3 Jack RJ45, J4 Jack RJ45, J5 Jack RJ45, J6 Jack RJ45, J7 Jack RJ45, J8 Jack RJ45, J9 DB142V-5.08-2P

Commit message: Revision for manufacturing
Parts:
- added FID1, FID2, FID3: Fiducial, Fiducial:Fiducial_1mm_Mask2mm, symbol Mechanical:Fiducial
Changed lines of the file:
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@@
+	)
+	(symbol
+		(lib_id "Mechanical:Fiducial")
+		(at 260.35 25.4 0)
+		(unit 1)
+		(exclude_from_sim no)
+		(in_bom no)
+		(on_board yes)
+		(dnp no)
+		(fields_autoplaced yes)
+		(property "Reference" "FID2"
+			(at 262.89 24.1299 0)
+			(effects
+				(font
+					(size 1.27 1.27)
+				)
+				(justify left)
+			)
+		)
+		(property "Value" "Fiducial"
+			(at 262.89 26.6699 0)
+			(effects
+				(font
+					(size 1.27 1.27)
+				)
+				(justify left)
+			)
+		)
+		(property "Footprint" "Fiducial:Fiducial_1mm_Mask2mm"
+			(at 260.35 25.4 0)
+			(effects
+				(font
+					(size 1.27 1.27)
+				)
+				(hide yes)
+			)
+		)
+		(property "Datasheet" "~"
+			(at 260.35 25.4 0)
+			(effects
+				(font
+					(size 1.27 1.27)
+				)
+				(hide yes)
+			)
+		)
+		(property "Description" "Fiducial Marker"
+			(at 260.35 25.4 0)
+			(effects
+				(font
+					(size 1.27 1.27)
+				)
+				(hide yes)
+			)
+		)
+		(instances
+			(project ""
+				(path "/e63e39d7-6ac0-4ffd-8aa3-1841a4541b55"
+					(reference "FID2")
+					(unit 1)
+				)
+			)
+		)
 	)
 	(symbol
@@
 	)
 	(symbol
+		(lib_id "Mechanical:Fiducial")
+		(at 260.35 19.05 0)
+		(unit 1)
+		(exclude_from_sim no)
+		(in_bom no)
+		(on_board yes)
+		(dnp no)
+		(fields_autoplaced yes)
+		(property "Reference" "FID1"
+			(at 262.89 17.7799 0)
+			(effects
+				(font
+					(size 1.27 1.27)
+				)
+				(justify left)
+			)
+		)
+		(property "Value" "Fiducial"
+			(at 262.89 20.3199 0)
+			(effects
+				(font
+					(size 1.27 1.27)
+				)
+				(justify left)
+			)
+		)
+		(property "Footprint" "Fiducial:Fiducial_1mm_Mask2mm"
+			(at 260.35 19.05 0)
+			(effects
+				(font
+					(size 1.27 1.27)
+				)
+				(hide yes)
+			)
+		)
+		(property "Datasheet" "~"
+			(at 260.35 19.05 0)
+			(effects
+				(font
+					(size 1.27 1.27)
+				)
+				(hide yes)
+			)
+		)
+		(property "Description" "Fiducial Marker"
+			(at 260.35 19.05 0)
+			(effects
+				(font
+					(size 1.27 1.27)
+				)
+				(hide yes)
+			)
+		)
+		(instances
+			(project ""
+				(path "/e63e39d7-6ac0-4ffd-8aa3-1841a4541b55"
+					(reference "FID1")
+					(unit 1)
+				)
+			)
+		)
+	)
+	(symbol
 		(lib_id "Connector_Generic:Conn_01x06")
 		(at 212.09 125.73 0)
@@
 					(unit 1)
 				)
+			)
+		)
+	)
+	(symbol
+		(lib_id "Mechanical:Fiducial")
+		(at 260.35 31.75 0)
+		(unit 1)
+		(exclude_from_sim no)
+		(in_bom no)
+		(on_board yes)
+		(dnp no)
+		(fields_autoplaced yes)
+		(property "Reference" "FID3"
+			(at 262.89 30.4799 0)
+			(effects
+				(font
+					(size 1.27 1.27)
+				)
+				(justify left)
+			)
+		)
+		(property "Value" "Fiducial"
+			(at 262.89 33.0199 0)
+			(effects
+				(font
+					(size 1.27 1.27)
+				)
+				(justify left)
+			)
+		)
+		(property "Footprint" "Fiducial:Fiducial_1mm_Mask2mm"
+			(at 260.35 31.75 0)
+			(effects
+				(font
+					(size 1.27 1.27)
+				)
+				(hide yes)
+			)
+		)
+		(property "Datasheet" "~"
+			(at 260.35 31.75 0)
+			(effects
+				(font
+					(size 1.27 1.27)
+				)
+				(hide yes)
+			)
+		)
+		(property "Description" "Fiducial Marker"
+			(at 260.35 31.75 0)
+			(effects
+				(font
+					(size 1.27 1.27)
+				)
+				(hide yes)
+			)
+		)
+		(instances
+			(project ""
+				(path "/e63e39d7-6ac0-4ffd-8aa3-1841a4541b55"
+					(reference "FID3")
+					(unit 1)
+				)

Commit message: Revising before production
Connections:
- net +24V: now reaches J1.1, J1.2, J2.1, J2.2, J3.1, J3.2, J4.1, J4.2, J5.1, J5.2, J6.1, J6.2, J7.1, J7.2, J8.1, J8.2, J9.1 (Pin_1), J9.2 (Pin_2)
- net CH4PAR2: now reaches J11.4 (Pin_4), J4.3, J4.6
- net CH4PAR3: now reaches J11.5 (Pin_5), J4.4, J4.5
- net CH4PAR4: now reaches J11.6 (Pin_6), J4.7, J4.8
- net CH3PAR2: now reaches J11.1 (Pin_1), J3.3, J3.6
- net CH3PAR3: now reaches J11.2 (Pin_2), J3.4, J3.5
- net CH3PAR4: now reaches J11.3 (Pin_3), J3.7, J3.8
- net CH2PAR2: now reaches J10.4 (Pin_4), J2.3, J2.6
- net CH2PAR3: now reaches J10.5 (Pin_5), J2.4, J2.5
- net CH2PAR4: now reaches J10.6 (Pin_6), J2.7, J2.8
- net CH1PAR2: now reaches J1.3, J1.6, J10.1 (Pin_1)
- net CH1PAR3: now reaches J1.4, J1.5, J10.2 (Pin_2)
- net CH1PAR4: now reaches J1.7, J1.8, J10.3 (Pin_3)
- net CH8PAR2: now reaches J13.4 (Pin_4), J8.3, J8.6
- net CH8PAR3: now reaches J13.5 (Pin_5), J8.4, J8.5
- net CH8PAR4: now reaches J13.6 (Pin_6), J8.7, J8.8
- net CH7PAR2: now reaches J13.1 (Pin_1), J7.3, J7.6
- net CH7PAR3: now reaches J13.2 (Pin_2), J7.4, J7.5
- net CH7PAR4: now reaches J13.3 (Pin_3), J7.7, J7.8
- net CH6PAR2: now reaches J12.4 (Pin_4), J6.3, J6.6
- net CH6PAR3: now reaches J12.5 (Pin_5), J6.4, J6.5
- net CH6PAR4: now reaches J12.6 (Pin_6), J6.7, J6.8
- net CH5PAR2: now reaches J12.1 (Pin_1), J5.3, J5.6
- net CH5PAR3: now reaches J12.2 (Pin_2), J5.4, J5.5
- net CH5PAR4: now reaches J12.3 (Pin_3), J5.7, J5.8
Other:
- moved on the sheet: J10, J11, J12, J13
