File: V3/rj45-breakout-8ch-v3.kicad_pcb (KiCad board)
At the start: 2 copper layers, 93 x 67.8 mm, 13 parts, among them J1 Jack RJ45, J10 DB141V-2.54-6P, J11 DB141V-2.54-6P, J12 DB141V-2.54-6P, J13 DB141V-2.54-6P, J2 Jack RJ45, J3 Jack RJ45, J4 Jack RJ45, J5 Jack RJ45, J6 Jack RJ45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

Commit message: Revision for manufacturing
Parts:
- added FID1: Fiducial, Fiducial:Fiducial_1mm_Mask2mm, F.Cu at (102.0, 64.5)
- added FID2: Fiducial, Fiducial:Fiducial_1mm_Mask2mm, F.Cu at (190.8, 64.5)
- added FID3: Fiducial, Fiducial:Fiducial_1mm_Mask2mm, F.Cu at (190.9, 128.0)
Routing:
- net Net-(J9-Pin_1): track 252.7 -> 0.00 mm
Other:
- rule pad_to_mask_clearance: 0 -> 0.1

Commit message: Small updates before fabrication
Parts:
- moved FID2 97.4 mm to (104.2, 109.2)
- moved FID3 21.4 mm to (180.5, 109.2)
- moved FID1 3.55 mm to (104.2, 67.2)
Routing:
- net Net-(J10-Pin_4): track 76.7 -> 59.7 mm
- net Net-(J10-Pin_1): track 56.4 -> 39.4 mm
- net Net-(J13-Pin_4): track 75.2 -> 58.2 mm
- net Net-(J13-Pin_1): track 53.3 -> 36.3 mm
- net Net-(J11-Pin_4): track 75.7 -> 58.7 mm
- net Net-(J12-Pin_1): track 54.3 -> 37.3 mm
- net Net-(J11-Pin_1): track 55.4 -> 38.3 mm
- net Net-(J12-Pin_4): track 74.7 -> 57.6 mm
- net Net-(J13-Pin_5): track 59.0 -> 55.9 mm
- net Net-(J13-Pin_2): track 37.5 -> 34.5 mm
- net Net-(J12-Pin_5): track 58.9 -> 55.8 mm
- net Net-(J12-Pin_2): track 38.6 -> 35.5 mm
- net Net-(J11-Pin_5): track 59.9 -> 56.9 mm
- net Net-(J11-Pin_2): track 39.6 -> 36.5 mm
- net Net-(J10-Pin_6): track 61.5 -> 58.4 mm
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